File: pmi-hw-carlos.sch (KiCad schematic (older format))
At the start: 19 parts, among them J1 Pmod-Interface-GPIO12, J2 Pmod-Interface-GPIO12, J3 Ground, J4 JumperBridge, SW1 Button1, SW2 Button2

Commit message: Update rescue lib
Parts:
- H1, H2, H3: symbol Mechanical-emt:Silkscreen_Label -> pmi-hw-carlos-rescue:Silkscreen_Label-Mechanical-emt
- J1, J2: symbol Pmod-Interface-emt:Pmod-Interface-GPIO12 -> pmi-hw-carlos-rescue:Pmod-Interface-GPIO12-Pmod-Interface-emt
Changed lines of the file:
@@
 $EndDescr
 $Comp
-L Pmod-Interface-emt:Pmod-Interface-GPIO12 J1
+L pmi-hw-carlos-rescue:Pmod-Interface-GPIO12-Pmod-Interface-emt J1
 U 1 1 6086BFD4
 P 950 1600
@@
 $EndComp
 $Comp
-L Pmod-Interface-emt:Pmod-Interface-GPIO12 J2
+L pmi-hw-carlos-rescue:Pmod-Interface-GPIO12-Pmod-Interface-emt J2
 U 1 1 6086C05D
 P 2650 1600
@@
 $EndComp
 $Comp
-L Mechanical-emt:Silkscreen_Label H1
+L pmi-hw-carlos-rescue:Silkscreen_Label-Mechanical-emt H1
 U 1 1 60893C8D
 P 2550 3750
@@
 $EndComp
 $Comp
-L Mechanical-emt:Silkscreen_Label H2
+L pmi-hw-carlos-rescue:Silkscreen_Label-Mechanical-emt H2
 U 1 1 60895E1B
 P 2550 4150
@@
 $EndComp
 $Comp
-L Mechanical-emt:Silkscreen_Label H3
+L pmi-hw-carlos-rescue:Silkscreen_Label-Mechanical-emt H3
 U 1 1 608960E2
 P 2550 3950
