File: pmi-hw-carlos.kicad_pcb (KiCad board)
At the start: 2 copper layers, 54.6 x 20.3 mm, 19 parts, among them J1 Pmod-Interface-GPIO12, J2 Pmod-Interface-GPIO12, J3 Ground, J4 JumperBridge, SW1 Button1, SW2 Button1

Commit message: Move project to Kicad 6, change load resistance R1 to 1k
Parts:
- R1: value 10k -> 1k
- SW2: value Button1 -> Button2
Connections:
- net +3V3 renamed +3.3V
- net /~BUTTON_1 renamed /~{BUTTON_1}
- net /~BUTTON_2 renamed /~{BUTTON_2}
Other:
- net class Default removed
- net class Supply removed

Commit message: Bump to version 1.2
Parts:
- SW1: value Button1 -> SW_Push; footprint Button_Switch-emt:SW_SPST_SCHURTER_1301.93XX -> Button_Switch-emt:SW_SPST_Schurter_1301.93XX
- SW2: value Button2 -> SW_Push; footprint Button_Switch-emt:SW_SPST_SCHURTER_1301.93XX -> Button_Switch-emt:SW_SPST_Schurter_1301.93XX
- renumbered H3 to H2, H2 to H3, R2 to R1, R3 to R2, R1 to R3, TP3 to TP1, TP4 to TP2, TP1 to TP3, TP2 to TP4
Routing:
- net /~{BUTTON_2}: track 53.2 -> 50.2 mm
- net /C_SUPP: track 56.0 -> 53.2 mm
- net /C_MEAS: track 54.5 -> 52.9 mm
- net /~{BUTTON_1}: track 65.6 -> 64.3 mm
- net GND: vias 30 -> 31
Other:
- outline, holes or cut-outs redrawn
- board text added: "PMI-CARLOS V1.2 2023"
- board text removed: "PMI-CARLOS V1.1 2021"
