File: pmi-hw-carlos.kicad_sch (KiCad schematic)
At the start: 19 parts, among them J1 Pmod-Interface-GPIO12, J2 Pmod-Interface-GPIO12, J3 Ground, J4 JumperBridge, SW1 Button1, SW2 Button2

Commit message: Bump to version 1.2
Parts:
- removed SW1: Button1, Button_Switch-emt:SW_SPST_SCHURTER_1301.93XX, symbol Switch:SW_DIP_x01
- removed SW2: Button2, Button_Switch-emt:SW_SPST_SCHURTER_1301.93XX, symbol Switch:SW_DIP_x01
- added SW1, SW2: SW_Push, Button_Switch-emt:SW_SPST_Schurter_1301.93XX, symbol Switch:SW_Push
- renumbered H3 to H2, H2 to H3, R2 to R1, R3 to R2, R1 to R3, TP3 to TP1, TP4 to TP2, TP1 to TP3, TP2 to TP4
Connections:
- net GND: now also SW1.1, SW2.1
- net ~{BUTTON_1}: now also SW1.2
- net ~{BUTTON_2}: now also SW2.2
Other:
- note added: "C charge/discharge"
- note added: "Pmod Connectors"
- note added: "Power"
- note removed: "C charge / discharge"
- note removed: "P-Interface"
